File: Hardware/_Sub_HW_EPen/v1_20231122/Design Folder/_HW_EPen/_autosave-_HW_EPen.kicad_pcb (KiCad board)
At the start: 2 copper layers, 49.5 x 29.2 mm, 50 parts, among them J301 HDR_4POS_VERT, J401 RECEPT_8POS_RA, J601 USB_microB_RA, U301 PIC16F15223_8BIT, U401 SN74HCS365PWR, U501 FT230XQ-R, U701 MIC5365-3.0YC5-TR

Commit message: Working on PCB layout
Parts:
- moved C507 5.08 mm to (100.8, 135.9)
- moved C506 4.77 mm to (100.8, 140.7)
- moved U501 0.75 mm to (100.3, 147.2)
Changed lines of the file:
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@@
   (net 52 "unconnected-(U701-NC-Pad4)")
   (footprint "Capacitor_SMD:C_0402_1005Metric" (layer "F.Cu")
-    (at 100.81 140.97)
+    (at 100.81 135.89)
     (descr "Capacitor SMD 0402 (1005 Metric), square (rectangular) end terminal, IPC_7351 nominal, (Body size source: IPC-SM-782 page 76, https://www.pcb-3d.com/wordpress/wp-content/uploads/ipc-sm-782a_amendment_1_and_2.pdf), generated with kicad-footprint-generator")
     (tags "capacitor")
@@
   )
   (footprint "Package_DFN_QFN:QFN-16-1EP_4x4mm_P0.65mm_EP2.1x2.1mm_ThermalVias" (layer "F.Cu")
-    (at 100.33 147.955 180)
+    (at 100.33 147.205 180)
     (descr "QFN, 16 Pin (http://www.thatcorp.com/datashts/THAT_1580_Datasheet.pdf), generated with kicad-footprint-generator ipc_noLead_generator.py")
     (tags "QFN NoLead")
@@
   )
   (footprint "Capacitor_SMD:C_0402_1005Metric" (layer "F.Cu")
-    (at 100.81 135.89)
+    (at 100.81 140.66)
     (descr "Capacitor SMD 0402 (1005 Metric), square (rectangular) end terminal, IPC_7351 nominal, (Body size source: IPC-SM-782 page 76, https://www.pcb-3d.com/wordpress/wp-content/uploads/ipc-sm-782a_amendment_1_and_2.pdf), generated with kicad-footprint-generator")
     (tags "capacitor")
