File: Hardware/_Sub_HW_EPen/v1_20231122/Design Folder/_HW_EPen/[04] - OUTPUT.kicad_sch (KiCad schematic)
At the start: 0 parts

Commit message: Working on Epen Schematic
Parts:
- added C401: 4u7F_16V, Capacitor_SMD:C_0805_2012Metric, symbol _SCHLIB_EPen:CAP_4.7uF_16V_X7R_C0805
- added C402: 10nF_50V, Capacitor_SMD:C_0402_1005Metric, symbol _SCHLIB_EPen:CAP_10nF_50V_X7R_C0402
- added J401: RECEPT_8POS_RA, Connector_PinSocket_2.54mm:PinSocket_1x08_P2.54mm_Horizontal, symbol _SCHLIB_EPen:CONN_RECEPT_8POS_1RAW_RA_2.54mm
- added R401, R403, R404, R405, R406, R407: 27R_1/16W_1%, Resistor_SMD:R_0402_1005Metric, symbol _SCHLIB_EPen:RES_27R_1/16W_1%_R0402
- added R402: 10kR_1/16W_1%, Resistor_SMD:R_0402_1005Metric, symbol _SCHLIB_EPen:RES_10kR_1/16W_1%_R0402
- added U401: SN74HCS365PWR, Package_SO:TSSOP-16_4.4x5mm_P0.65mm, symbol _SCHLIB_EPen:IC_BUFFER_SN74HCS365PWR_NON-INV_6BIT_16-TSSOP
Connections:
- new net: R405.1, U401.9 (Y4)
- new net: R406.1, U401.11 (Y5)
- new net: R407.1, U401.13 (Y6)
- new net: R401.1, U401.3 (Y1)
- new net: R404.1, U401.5 (Y2)
- new net A1: U401.2 (A1)
- new net A2: U401.4 (A2)
- new net A3: R403.1, U401.6 (A3)
- new net A4: U401.10 (A4)
- new net A5: U401.12 (A5)
- new net A6: U401.14 (A6)
- new net EEPROM_~{WP}: J401.6, R406.2
- new net GND: C401.2, C402.2, J401.1, J401.8, U401.8 (GND)
- new net MCU_~{MCLR}: J401.7, R407.2
- new net SPI_CS: J401.2, R401.2
- new net SPI_MISO: J401.3, R403.2
- new net SPI_MOSI: J401.4, R404.2
- new net SPI_SCK: J401.5, R405.2
- new net VIN: C401.1, C402.1, R402.1, U401.16 (VCC)
- new net Y3: U401.7 (Y3)
- new net ~{EN}: R402.2, U401.1 (~{OE}), U401.15 (~{OE2})
Other:
- note added: "DESIGN NOTE:"
- note added: "Imax ~= 7mA"
- note added: "TWO CONFIG IS POSSIBLE SPI_CS | MCU_~{MCLR} SPI_MISO | EEPROM_~{WP} SPI_MOSI | SPI_SCK SPI_SCK | SPI_MOSI EEPROM_~{WP} | SPI_MISO MCU_~{MCLR} | SPI_CS If the connector has been attached in reverse There will be no damage to the device, the only problem is that The user need to connect it in the correct way!"
- note added: "UNCHECKED"

Commit message: More progress on EPen Hardware
Other:
- note removed: "UNCHECKED"
- company: (none) -> mend0z0
Changed lines of the file:
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@@
 (kicad_sch (version 20230121) (generator eeschema)
   (paper "B")
+  (title_block
+    (company "mend0z0")
+    (comment 1 "v1.0")
+    (comment 2 "PRELIMINARY")
+    (comment 4 "_BOM_EPen.html")
+    (comment 5 "_HW_EPen.pcb")
+    (comment 6 "_GBR_EPen.zip")
+    (comment 7 "_BOM_EPen.html")
+    (comment 9 "First Release")
+  )
   (junction (at 153.67 158.75) (diameter 0) (color 0 0 0 0)
   )
@@
     (effects (font (size 1.27 1.27)) (justify left bottom))
   )
-  (text "UNCHECKED" (at 370.84 35.56 0)
-    (effects (font (size 5.08 5.08) (thickness 1.016) bold) (justify left bottom))
-  )
   (text "Imax ~= 7mA" (at 208.28 116.84 0)

Commit message: _HW_EPen is ready to be worked for layout
Parts:
- C401, C402, J401, R401, R402, R403, R404, R405, R406, R407, U401: SCH CHECK SCH (N/A) -> SCH (CHECKED)
Connections:
- net A3 renamed SN74HCS365_A3
Other:
- note added: "INFO:"
- note added: "LAYOUT NOTE:"
- title: (none) -> _HW_EPen
- moved on the sheet: C401, C402, R402, U401

Commit message: Updating file templates and structures...
Other:
- moved on the sheet: C401, C402, J401, R401, R402, R403, R404, R405, R406, R407, U401

Commit message: Updating Hardware File structures
Parts:
- C401: Manufacturer (none) -> Murata Electronics; Part Number GRM21BR71C475KE51L -> (none); Part Number (Manufacturer) (none) -> GRM21BR71C475KE51L; Part Number (Vendor) (none) -> 490-14466-2-ND; Vendor (none) -> Digikey
- C402: Manufacturer (none) -> Samsung Electro-Mechanics; Part Number CL05B103KB5NNNC -> (none); Part Number (Manufacturer) (none) -> CL05B103KB5NNNC; Part Number (Vendor) (none) -> 1276-1028-2-ND; Vendor (none) -> Digikey
- J401: Manufacturer (none) -> Samtec Inc.; Part Number SSQ-108-02-T-S-RA -> (none); Part Number (Manufacturer) (none) -> SSQ-108-02-T-S-RA; Part Number (Vendor) (none) -> SAM1195-08-ND; Vendor (none) -> Digikey
- R401, R403, R404, R405, R406, R407: Manufacturer (none) -> Bourns Inc.; Part Number CR0402-FX-27R0GLF -> (none); Part Number (Manufacturer) (none) -> CR0402-FX-27R0GLF; Part Number (Vendor) (none) -> CR0402-FX-27R0GLFTR-ND; Vendor (none) -> Digikey
- R402: Manufacturer (none) -> Bourns Inc.; Part Number CR0402-FX-1002GLF -> (none); Part Number (Manufacturer) (none) -> CR0402-FX-1002GLF; Part Number (Vendor) (none) -> CR0402-FX-1002GLFTR-ND; Vendor (none) -> Digikey
- U401: Manufacturer (none) -> Texas Instruments; Part Number SN74HCS365PWR -> (none); Part Number (Manufacturer) (none) -> SN74HCS365PWR; Part Number (Vendor) (none) -> 296-SN74HCS365PWRTR-ND; Vendor (none) -> Digikey
