File: Hardware/_Sub_HW_EPen/v1_20231122/Design Folder/_HW_EPen/[05] - FT230X_DRIVER.kicad_sch (KiCad schematic)
At the start: 13 parts, among them U501 FT230XQ-R

Commit message: More progress on EPen Hardware
Other:
- note removed: "UNCHECKED"
- company: (none) -> mend0z0
Changed lines of the file:
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@@
 (kicad_sch (version 20230121) (generator eeschema)
   (paper "B")
+  (title_block
+    (company "mend0z0")
+    (comment 1 "v1.0")
+    (comment 2 "PRELIMINARY")
+    (comment 4 "_BOM_EPen.html")
+    (comment 5 "_HW_EPen.pcb")
+    (comment 6 "_GBR_EPen.zip")
+    (comment 7 "_BOM_EPen.html")
+    (comment 9 "First Release")
+  )
   (junction (at 184.15 149.86) (diameter 0) (color 0 0 0 0)
   )
@@
     (fill (type none))
   )
-  (text "UNCHECKED" (at 369.57 38.1 0)
-    (effects (font (size 5.08 5.08) (thickness 1.016) bold) (justify left bottom))
-  )
   (text "I ~= 50mA" (at 234.95 137.16 0)

Commit message: _HW_EPen is ready to be worked for layout
Parts:
- C501, C502, C503, C504, C505, C506, C507, R501, R502, R503, R504, R505, U501: SCH CHECK SCH (N/A) -> SCH (CHECKED)
Other:
- title: (none) -> _HW_EPen
Changed lines of the file:
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@@
   (paper "B")
   (title_block
+    (title "_HW_EPen")
+    (date "2023-11-28")
+    (rev "v1.0")
     (company "mend0z0")
     (comment 1 "v1.0")
-    (comment 2 "PRELIMINARY")
+    (comment 2 "CHECKED")
     (comment 4 "_BOM_EPen.html")
     (comment 5 "_HW_EPen.pcb")
     (comment 6 "_GBR_EPen.zip")
     (comment 7 "_BOM_EPen.html")
+    (comment 8 "N/A")
     (comment 9 "First Release")
   )
@@
       (effects (font (size 1.27 1.27)))
     )
-    (property "SCH CHECK" "SCH (N/A)" (at 203.2 105.41 0)
+    (property "SCH CHECK" "SCH (CHECKED)" (at 203.2 105.41 0)
       (effects (font (size 1.27 1.27)))
     )
@@
     (pin "12")
     (pin "1")
+    (pin "16")
     (instances
       (project "_HW_EPen"
@@
       (effects (font (size 1.27 1.27)))
     )
-    (property "SCH CHECK" "SCH (N/A)" (at 265.43 110.49 0)
+    (property "SCH CHECK" "SCH (CHECKED)" (at 265.43 110.49 0)
       (effects (font (size 1.27 1.27)))
     )
@@
       (effects (font (size 1.27 1.27)) (justify left))
     )
-    (property "SCH CHECK" "SCH (N/A)" (at 156.21 151.13 90)
+    (property "SCH CHECK" "SCH (CHECKED)" (at 156.21 151.13 90)
       (effects (font (size 1.27 1.27)) (justify left))
     )
@@
       (effects (font (size 1.27 1.27)) (justify left))
     )
-    (property "SCH CHECK" "SCH (N/A)" (at 64.77 113.03 90)
+    (property "SCH CHECK" "SCH (CHECKED)" (at 64.77 113.03 90)
       (effects (font (size 1.27 1.27)) (justify left))
     )
@@
       (effects (font (size 1.27 1.27)))
     )
-    (property "SCH CHECK" "SCH (N/A)" (at 265.43 120.65 0)
+    (property "SCH CHECK" "SCH (CHECKED)" (at 265.43 120.65 0)
       (effects (font (size 1.27 1.27)))
     )
@@
       (effects (font (size 1.27 1.27)))
     )
-    (property "SCH CHECK" "SCH (N/A)" (at 151.13 93.98 0)
+    (property "SCH CHECK" "SCH (CHECKED)" (at 151.13 93.98 0)
       (effects (font (size 1.27 1.27)))
     )
@@
       (effects (font (size 1.27 1.27)) (justify left))
     )
-    (property "SCH CHECK" "SCH (N/A)" (at 114.3 105.41 90)
+    (property "SCH CHECK" "SCH (CHECKED)" (at 114.3 105.41 90)
       (effects (font (size 1.27 1.27)) (justify left))
     )
@@
       (effects (font (size 1.27 1.27)) (justify left))
     )
-    (property "SCH CHECK" "SCH (N/A)" (at 227.33 151.13 90)
+    (property "SCH CHECK" "SCH (CHECKED)" (at 227.33 151.13 90)
       (effects (font (size 1.27 1.27)) (justify left))
     )
@@
       (effects (font (size 1.27 1.27)) (justify left))
     )
-    (property "SCH CHECK" "SCH (N/A)" (at 64.77 130.81 90)
+    (property "SCH CHECK" "SCH (CHECKED)" (at 64.77 130.81 90)
       (effects (font (size 1.27 1.27)) (justify left))
     )
@@
       (effects (font (size 1.27 1.27)) (justify left))
     )
-    (property "SCH CHECK" "SCH (N/A)" (at 97.79 105.41 90)
+    (property "SCH CHECK" "SCH (CHECKED)" (at 97.79 105.41 90)
       (effects (font (size 1.27 1.27)) (justify left))
     )
@@
       (effects (font (size 1.27 1.27)) (justify left))
     )
-    (property "SCH CHECK" "SCH (N/A)" (at 138.43 151.13 90)
+    (property "SCH CHECK" "SCH (CHECKED)" (at 138.43 151.13 90)
       (effects (font (size 1.27 1.27)) (justify left))
     )
@@
       (effects (font (size 1.27 1.27)))
     )
-    (property "SCH CHECK" "SCH (N/A)" (at 151.13 86.36 0)
+    (property "SCH CHECK" "SCH (CHECKED)" (at 151.13 86.36 0)
       (effects (font (size 1.27 1.27)))
     )
@@
       (effects (font (size 1.27 1.27)) (justify left))
     )
-    (property "SCH CHECK" "SCH (N/A)" (at 120.65 151.13 90)
-      (effects (font (size 1.27 1.27)) (justify left))
-    )
+    (property "SCH CHECK" "SCH (CHECKED)" (at 120.65 151.13 90)
+      (effects (font (size 1.27 1.27)) (justify left))
+    )

Commit message: Working on PCB layout
Connections:
- no-connect marks 5 -> 6
Changed lines of the file:
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@@
   (junction (at 135.89 157.48) (diameter 0) (color 0 0 0 0)
   )
-  (no_connect (at 224.79 125.73))
-  (no_connect (at 224.79 130.81))
+  (no_connect (at 224.79 127))
+  (no_connect (at 224.79 132.08))
+  (no_connect (at 224.79 121.92))
   (no_connect (at 224.79 119.38))
-  (no_connect (at 224.79 133.35))
-  (no_connect (at 224.79 128.27))
+  (no_connect (at 224.79 134.62))
+  (no_connect (at 224.79 129.54))
   (wire (pts (xy 146.05 85.09) (xy 161.29 85.09))
     (stroke (width 0) (type default))
@@
     (stroke (width 0) (type default))
   )
-  (wire (pts (xy 224.79 125.73) (xy 220.98 125.73))
+  (wire (pts (xy 224.79 127) (xy 220.98 127))
     (stroke (width 0) (type default))
   )
@@
     (stroke (width 0) (type default))
   )
+  (wire (pts (xy 224.79 121.92) (xy 220.98 121.92))
+    (stroke (width 0) (type default))
+  )
   (wire (pts (xy 220.98 113.03) (xy 229.87 113.03))
     (stroke (width 0) (type default))
   )
-  (wire (pts (xy 224.79 133.35) (xy 220.98 133.35))
+  (wire (pts (xy 224.79 134.62) (xy 220.98 134.62))
     (stroke (width 0) (type default))
   )
@@
     (stroke (width 0) (type default))
   )
-  (wire (pts (xy 224.79 128.27) (xy 220.98 128.27))
+  (wire (pts (xy 224.79 129.54) (xy 220.98 129.54))
     (stroke (width 0) (type default))
   )
@@
     (stroke (width 0) (type default))
   )
-  (wire (pts (xy 224.79 130.81) (xy 220.98 130.81))
+  (wire (pts (xy 224.79 132.08) (xy 220.98 132.08))
     (stroke (width 0) (type default))
   )

Commit message: Updating file templates and structures...
Other:
- moved on the sheet: C501, C502, C503, C504, C505, C506, C507, R501, R502, R503, R504, R505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

Commit message: Updating Hardware File structures
Parts:
- C501, C502, C505: Manufacturer (none) -> Murata Electronics; Part Number GRM155R71H104KE14J -> (none); Part Number (Manufacturer) (none) -> GRM155R71H104KE14J; Part Number (Vendor) (none) -> 490-13342-2-ND; Vendor (none) -> Digikey
- C503: Manufacturer (none) -> Murata Electronics; Part Number GRM21BR71C475KE51L -> (none); Part Number (Manufacturer) (none) -> GRM21BR71C475KE51L; Part Number (Vendor) (none) -> 490-14466-2-ND; Vendor (none) -> Digikey
- C504: Manufacturer (none) -> Samsung Electro-Mechanics; Part Number CL05B103KB5NNNC -> (none); Part Number (Manufacturer) (none) -> CL05B103KB5NNNC; Part Number (Vendor) (none) -> 1276-1028-2-ND; Vendor (none) -> Digikey
- C506, C507: Manufacturer (none) -> KEMET; Part Number C0402C470J5RACAUTO -> (none); Part Number (Manufacturer) (none) -> C0402C470J5RACAUTO; Part Number (Vendor) (none) -> 399-C0402C470J5RACAUTOTR-ND; Vendor (none) -> Digikey
- R501: Manufacturer (none) -> Bourns Inc.; Part Number CR0402-FX-1002GLF -> (none); Part Number (Manufacturer) (none) -> CR0402-FX-1002GLF; Part Number (Vendor) (none) -> CR0402-FX-1002GLFTR-ND; Vendor (none) -> Digikey
- R502, R503, R504, R505: Manufacturer (none) -> Bourns Inc.; Part Number CR0402-FX-27R0GLF -> (none); Part Number (Manufacturer) (none) -> CR0402-FX-27R0GLF; Part Number (Vendor) (none) -> CR0402-FX-27R0GLFTR-ND; Vendor (none) -> Digikey
- U501: Manufacturer (none) -> FTDI, Future Technology Devices International Ltd; Part Number FT230XQ-R -> (none); Part Number (Manufacturer) (none) -> FT230XQ-R; Part Number (Vendor) (none) -> 768-1130-2-ND; Vendor (none) -> Digikey
