File: Hardware/_Sub_HW_EPen/v1_20231122/Design Folder/_HW_EPen/[06] - USB.kicad_sch (KiCad schematic)
At the start: 0 parts

Commit message: Working on Epen Schematic
Parts:
- added C601: 100nF_50V, Capacitor_SMD:C_0402_1005Metric, symbol _SCHLIB_EPen:CAP_100nF_50V_X7R_C0402
- added D601, D602, D603: TVS_6.5V_3A, symbol _SCHLIB_EPen:TVS_5V(MAX)_6.5(Vbr-min)_3A(8/20us)_SOD882
- added F601, F602, F603: 100mA_15V_0.5R, Fuse:Fuse_0603_1608Metric, symbol _SCHLIB_EPen:FUSE_100mA(Ih)_250mA(It)_15V_0.5Ohm_F0603
- added J601: USB_microB_RA, Connector_USB:USB_Micro-B_Amphenol_10118194_Horizontal, symbol _SCHLIB_EPen:CONN_RECEPT_USB2.0_microB_5POS_RA
- added LED601: RED_2V, LED_SMD:LED_0402_1005Metric, symbol _SCHLIB_EPen:LED_RED_2V_624nm_LED0402
- added R601: 470R_1/16W_1%, Resistor_SMD:R_0402_1005Metric, symbol _SCHLIB_EPen:RES_470R_1/16W_1%_R0402
Connections:
- new net: LED601.2, R601.2
- new net: F601.1, J601.1 (VBUS)
- new net D+: F602.1, J601.3 (D+)
- new net D-: F603.1, J601.2 (D-)
- new net Earth: J601.6 (SH)
- new net GND: C601.2, D601.2, D602.2, D603.2, J601.5 (GND), LED601.1
- new net USBDM: D603.1, F603.2
- new net USBDP: D602.1, F602.2
- new net VBUS: C601.1, D601.1, F601.2, R601.1
- no-connect marks 0 -> 1
Other:
- note added: "I ~= 100mA"
- note added: "I ~= 6mA"
- note added: "UNCHECKED"

Commit message: More progress on EPen Hardware
Other:
- note removed: "UNCHECKED"
- company: (none) -> mend0z0
Changed lines of the file:
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@@
 (kicad_sch (version 20230121) (generator eeschema)
   (paper "B")
+  (title_block
+    (company "mend0z0")
+    (comment 1 "v1.0")
+    (comment 2 "PRELIMINARY")
+    (comment 4 "_BOM_EPen.html")
+    (comment 5 "_HW_EPen.pcb")
+    (comment 6 "_GBR_EPen.zip")
+    (comment 7 "_BOM_EPen.html")
+    (comment 9 "First Release")
+  )
   (junction (at 200.66 80.01) (diameter 0) (color 0 0 0 0)
   )
@@
   (junction (at 241.3 80.01) (diameter 0) (color 0 0 0 0)
   )
-  (no_connect (at 146.05 132.08))
+  (no_connect (at 142.24 132.08))
   (wire (pts (xy 200.66 152.4) (xy 200.66 154.94))
     (stroke (width 0) (type default))
@@
     (stroke (width 0) (type default))
   )
-  (wire (pts (xy 146.05 132.08) (xy 138.43 132.08))
+  (wire (pts (xy 142.24 132.08) (xy 138.43 132.08))
     (stroke (width 0) (type default))
   )
@@
     (fill (type none))
   )
-  (text "UNCHECKED" (at 370.84 35.56 0)
-    (effects (font (size 5.08 5.08) (thickness 1.016) bold) (justify left bottom))
-  )
   (text "I ~= 100mA" (at 260.35 77.47 0)

Commit message: _HW_EPen is ready to be worked for layout
Parts:
- C601, F601, F602, F603, LED601, R601: SCH CHECK SCH (N/A) -> SCH (CHECKED)
- D601, D602, D603: footprint (none) -> _PCBLIB_EPen:CR_7PCT_L3F_TOS; SCH CHECK SCH (N/A) -> SCH (CHECKED)
- J601: Package (none) -> SMT - microB; SCH CHECK SCH (N/A) -> SCH (CHECKED)
Other:
- title: (none) -> _HW_EPen
- moved on the sheet: F602, F603

Commit message: Hardware is almost done
Parts:
- J601: footprint Connector_USB:USB_Micro-B_Amphenol_10118194_Horizontal -> _PCBLIB_EPen:USB_Micro-B_Amphenol_10118194_Horizontal
Changed lines of the file:
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@@
       (effects (font (size 1.27 1.27)))
     )
-    (property "Footprint" "Connector_USB:USB_Micro-B_Amphenol_10118194_Horizontal" (at 128.27 106.68 0)
+    (property "Footprint" "_PCBLIB_EPen:USB_Micro-B_Amphenol_10118194_Horizontal" (at 128.27 106.68 0)
       (effects (font (size 1.27 1.27)) (justify left) hide)
     )

Commit message: Updating file templates and structures...
Other:
- moved on the sheet: C601, D601, D602, D603, F601, F602, F603, J601, LED601, R601

Commit message: Updating Hardware File structures
Parts:
- C601: Manufacturer (none) -> Murata Electronics; Part Number GRM155R71H104KE14J -> (none); Part Number (Manufacturer) (none) -> GRM155R71H104KE14J; Part Number (Vendor) (none) -> 490-13342-2-ND; Vendor (none) -> Digikey
- D601, D602, D603: Manufacturer (none) -> Good-Ark Semiconductor; Part Number GSEWT5B003 -> (none); Part Number (Manufacturer) (none) -> GSEWT5B003; Part Number (Vendor) (none) -> 4786-GSEWT5B003TR-ND; Vendor (none) -> Digikey
- F601, F602, F603: Manufacturer (none) -> Eaton - Electronics Division; Part Number PTS060315V010 -> (none); Part Number (Manufacturer) (none) -> PTS060315V010; Part Number (Vendor) (none) -> 283-PTS060315V010TR-ND; Vendor (none) -> Digikey
- J601: Manufacturer (none) -> Amphenol ICC (FCI); Part Number 10118194-0001LF -> (none); Part Number (Manufacturer) (none) -> 10118194-0001LF; Part Number (Vendor) (none) -> 609-4618-2-ND; Vendor (none) -> Digikey
- LED601: Manufacturer (none) -> Harvatek Corporation; Part Number B2841USD-20D001014U1930 -> (none); Part Number (Manufacturer) (none) -> B2841USD-20D001014U1930; Part Number (Vendor) (none) -> 3147-B2841USD-20D001014U1930TR-ND; Vendor (none) -> Digikey
- R601: Manufacturer (none) -> Bourns Inc.; Part Number CR0402-FX-4700GLF -> (none); Part Number (Manufacturer) (none) -> CR0402-FX-4700GLF; Part Number (Vendor) (none) -> CR0402-FX-4700GLFTR-ND; Vendor (none) -> Digikey
