File: Hardware/_Sub_HW_EPen/v1_20231122/Design Folder/_HW_EPen/[08] - MECHANICAL PARTS.kicad_sch (KiCad schematic)
At the start: 0 parts

Commit message: EPen layout is almost done
Parts:
- added FD801, FD802: 1.5mmX3mm, Fiducial:Fiducial_1.5mm_Mask3mm, symbol _SCHLIB_EPen:MECH_PAD_FIDUCIAL_1.5mm_3mm
- added GR801: Mend0z0 Logo, _PCBLIB_EPen:LOGO_MEND0Z0, symbol _SCHLIB_EPen:MECH_GR_LOGO_MEND0Z0_TOP LAYER
- added MH801, MH802, MH803, MH804: M2.5_DIN965, MountingHole:MountingHole_2.7mm_M2.5_DIN965_Pad, symbol _SCHLIB_EPen:MECH_HOLE_MOUNTING_M2.5_DIN965_WITH NET
Connections:
- new net Earth: MH801.1, MH802.1, MH803.1, MH804.1

Commit message: Updating file templates and structures...
Other:
- moved on the sheet: FD801, FD802, GR801, MH801, MH802, MH803, MH804
