File: Hardware/_Sub_HW_EPen/v1_20231122/Design Folder/_HW_EPen/_HW_EPen.kicad_pcb (KiCad board)
At the start: 2 copper layers, 49.5 x 29.2 mm, 50 parts, among them J301 HDR_4POS_VERT, J401 RECEPT_8POS_RA, J601 USB_microB_RA, U301 PIC16F15223_8BIT, U401 SN74HCS365PWR, U501 FT230XQ-R, U701 MIC5365-3.0YC5-TR

Commit message: EPen layout is almost done
Parts:
- added FD801: 1.5mmX3mm, Fiducial:Fiducial_1.5mm_Mask3mm, F.Cu at (129.2, 126.5)
- added FD802: 1.5mmX3mm, Fiducial:Fiducial_1.5mm_Mask3mm, F.Cu at (98.6, 127.0)
- added GR801: Mend0z0 Logo, _PCBLIB_EPen:LOGO_MEND0Z0, F.Cu at (102.7, 128.7)
- added MH801: M2.5_DIN965, MountingHole:MountingHole_2.7mm_M2.5_DIN965_Pad, F.Cu at (91.5, 150.5)
- added MH802: M2.5_DIN965, MountingHole:MountingHole_2.7mm_M2.5_DIN965_Pad, F.Cu at (135.8, 150.4)
- added MH803: M2.5_DIN965, MountingHole:MountingHole_2.7mm_M2.5_DIN965_Pad, F.Cu at (135.8, 126.4)
- added MH804: M2.5_DIN965, MountingHole:MountingHole_2.7mm_M2.5_DIN965_Pad, F.Cu at (91.5, 126.4)
- moved C401 48.3 mm to (115.1, 149.1)
- moved C402 48.0 mm to (114.3, 151.1), turned to 180 degrees
- moved U401 36.8 mm to (121.9, 148.0), turned to 180 degrees
- moved R402 33.5 mm to (129.5, 150.2), turned to 180 degrees
- moved R701 27.3 mm to (106.9, 148.6), turned to 180 degrees
- moved R702 26.1 mm to (110.5, 151.1), turned to 180 degrees
- moved U701 25.5 mm to (110.5, 147.3)
- moved LED701 24.9 mm to (110.5, 149.9), turned to 180 degrees
- moved C701 22.5 mm to (106.9, 146.7), turned to 180 degrees
- moved C702 16.9 mm to (114.3, 146.7)
- moved LED301 14.2 mm to (116.5, 128.9), turned to 180 degrees
- moved C303 12.6 mm to (114.2, 128.9), turned to 0 degrees
- moved R504 12.6 mm to (111.9, 128.9)
- moved R505 12.1 mm to (110.6, 130.2)
- moved R303 11.3 mm to (116.5, 130.2)
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Routing:
- net Earth: track 0.00 -> 100.7 mm
- net /BLOCK DIAGRAM/LDO +3V0DC/+5VDC: track 0.00 -> 93.9 mm, vias 0 -> 6
- net /BLOCK DIAGRAM/MCU/PIC_ICSPDAT: track 0.00 -> 74.7 mm, vias 0 -> 3
- net GND: track 0.00 -> 53.5 mm, vias 0 -> 27
- net /BLOCK DIAGRAM/MCU/PIC_ICSPCLK: track 0.00 -> 52.5 mm, vias 0 -> 2
- net /BLOCK DIAGRAM/MCU/SPI_CS: track 0.00 -> 47.2 mm, vias 0 -> 2
- net /BLOCK DIAGRAM/LDO +3V0DC/MIC5365_PIN_EN: track 0.00 -> 32.8 mm, vias 0 -> 2
- net /BLOCK DIAGRAM/LDO +3V0DC/+3VDC: track 0.00 -> 31.9 mm
- net Net-(U501-TXD): track 0.00 -> 30.6 mm
- net /BLOCK DIAGRAM/MCU/SPI_MOSI: track 0.00 -> 28.3 mm, vias 0 -> 2
- net Net-(U401-Y6): track 0.00 -> 28.1 mm
- net Net-(U501-RXD): track 0.00 -> 24.0 mm, vias 0 -> 2
- net /BLOCK DIAGRAM/MCU/MCU_~{RESET}: track 0.00 -> 23.8 mm, vias 0 -> 2
- net Net-(U401-Y5): track 0.00 -> 23.8 mm
- net /BLOCK DIAGRAM/MCU/SPI_MISO: track 0.00 -> 20.8 mm, vias 0 -> 2
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- added copper zone on B.Cu, net GND
Other:
- outline, holes or cut-outs redrawn
- board text added: "GND ~{MCLR} ~{WP} SCK MOSI MISO CS GND"
- board text added: "PCB Layout"
- board text added: "PRELIMINARY"
- board text added: "_HW_EPen v1.0, 2023/11/28 DSN: SiavashTP"
- board text added: "~{MCLR} GND DAT CLK"

Commit message: Latest update
Routing:
- net /BLOCK DIAGRAM/FT230X_DRIVER/USBDM: track 10.2 -> 9.13 mm, vias 0 -> 2
- net /BLOCK DIAGRAM/FT230X_DRIVER/FT230X_3V3OUT: track 15.7 -> 15.2 mm
Changed lines of the file:
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@@
     (pts (xy 88.9 123.825) (xy 88.9 153.035))
     (height 19.05)
-    (gr_text "1150.0000 mils" (at 68.7 138.43 90) (layer "Dwgs.User")
+    (gr_text "29.2100 mm" (at 68.7 138.43 90) (layer "Dwgs.User")
       (effects (font (size 1 1) (thickness 0.15)))
     )
@@
     (pts (xy 88.9 153.035) (xy 138.43 153.035))
     (height 13.97)
-    (gr_text "1950.0000 mils" (at 113.665 165.855) (layer "Dwgs.User")
+    (gr_text "49.5300 mm" (at 113.665 165.855) (layer "Dwgs.User")
       (effects (font (size 1 1) (thickness 0.15)))
     )
@@
   (via (at 104.8505 148.971) (size 0.8) (drill 0.4) (layers "F.Cu" "B.Cu") (net 5))
   (via (at 99.568 142.24) (size 0.8) (drill 0.4) (layers "F.Cu" "B.Cu") (net 5))
-  (segment (start 100.965 144.526) (end 99.568 143.129) (width 0.25) (layer "B.Cu") (net 5))
+  (segment (start 104.14 146.812) (end 104.14 145.542) (width 0.25) (layer "B.Cu") (net 5))
+  (segment (start 101.854 144.526) (end 99.568 142.24) (width 0.25) (layer "B.Cu") (net 5))
   (segment (start 104.8505 147.5225) (end 104.14 146.812) (width 0.25) (layer "B.Cu") (net 5))
+  (segment (start 104.14 145.542) (end 103.124 144.526) (width 0.25) (layer "B.Cu") (net 5))
+  (segment (start 103.124 144.526) (end 101.854 144.526) (width 0.25) (layer "B.Cu") (net 5))
   (segment (start 104.8505 148.971) (end 104.8505 147.5225) (width 0.25) (layer "B.Cu") (net 5))
-  (segment (start 104.14 146.812) (end 104.14 145.542) (width 0.25) (layer "B.Cu") (net 5))
-  (segment (start 99.568 143.129) (end 99.568 142.24) (width 0.25) (layer "B.Cu") (net 5))
-  (segment (start 103.124 144.526) (end 100.965 144.526) (width 0.25) (layer "B.Cu") (net 5))
-  (segment (start 104.14 145.542) (end 103.124 144.526) (width 0.25) (layer "B.Cu") (net 5))
   (segment (start 98.354 147.63) (end 98.044 147.32) (width 0.25) (layer "F.Cu") (net 6))
   (segment (start 97 150.269) (end 97 147.32) (width 0.25) (layer "F.Cu") (net 6))
@@
   (segment (start 106.045 128.651) (end 105.156 129.54) (width 0.762) (layer "B.Cu") (net 6))
   (segment (start 96.647 138.938) (end 96.647 141.478) (width 0.762) (layer "B.Cu") (net 6))
-  (segment (start 97.663 146.05) (end 98.593 146.98) (width 0.25) (layer "F.Cu") (net 7))
-  (segment (start 98.593 146.98) (end 99.65 146.98) (width 0.25) (layer "F.Cu") (net 7))
+  (segment (start 97 146.05) (end 97.8154 146.05) (width 0.25) (layer "F.Cu") (net 7))
+  (segment (start 97.8154 146.05) (end 98.7454 146.98) (width 0.25) (layer "F.Cu") (net 7))
   (segment (start 97.03 146.02) (end 97 146.05) (width 0.25) (layer "F.Cu") (net 7))
+  (segment (start 98.7454 146.98) (end 99.65 146.98) (width 0.25) (layer "F.Cu") (net 7))
   (segment (start 97.03 144.78) (end 97.03 146.02) (width 0.25) (layer "F.Cu") (net 7))
-  (segment (start 97 146.05) (end 97.663 146.05) (width 0.25) (layer "F.Cu") (net 7))
-  (segment (start 101.6 141.73) (end 101.6 140.66) (width 0.25) (layer "F.Cu") (net 8))
+  (segment (start 102.235 141.8336) (end 101.6 141.1986) (width 0.25) (layer "F.Cu") (net 8))
+  (segment (start 102.235 142.365) (end 102.235 141.8336) (width 0.25) (layer "F.Cu") (net 8))
   (segment (start 99.339569 139.319069) (end 99.2125 139.192) (width 0.25) (layer "F.Cu") (net 8))
-  (segment (start 102.235 142.365) (end 101.6 141.73) (width 0.25) (layer "F.Cu") (net 8))
+  (segment (start 101.6 141.1986) (end 101.6 140.66) (width 0.25) (layer "F.Cu") (net 8))
   (segment (start 101.6 140.66) (end 101.6 139.319069) (width 0.25) (layer "F.Cu") (net 8))
   (segment (start 101.6 139.319069) (end 99.339569 139.319069) (width 0.25) (layer "F.Cu") (net 8))
+  (segment (start 101.6 138.2522) (end 101.6 137.16) (width 0.25) (layer "F.Cu") (net 9))
   (segment (start 101.6 137.16) (end 99.2125 137.16) (width 0.25) (layer "F.Cu") (net 9))
   (segment (start 101.6 135.89) (end 101.6 137.16) (width 0.25) (layer "F.Cu") (net 9))
-  (segment (start 100.965 142.365) (end 98.425 139.825) (width 0.25) (layer "F.Cu") (net 9))
-  (segment (start 98.425 139.825) (end 98.425 137.9475) (width 0.25) (layer "F.Cu") (net 9))
-  (segment (start 98.425 137.9475) (end 99.2125 137.16) (width 0.25) (layer "F.Cu") (net 9))
+  (segment (start 100.962952 141.543668) (end 100.965 141.545716) (width 0.25) (layer "F.Cu") (net 9))
+  (segment (start 100.965 141.545716) (end 100.965 142.365) (width 0.25) (layer "F.Cu") (net 9))
+  (via (at 100.962952 141.543668) (size 0.8) (drill 0.4) (layers "F.Cu" "B.Cu") (net 9))
+  (via (at 101.6 138.2522) (size 0.8) (drill 0.4) (layers "F.Cu" "B.Cu") (net 9))
+  (segment (start 100.962952 141.543668) (end 101.6 140.90662) (width 0.25) (layer "B.Cu") (net 9))
+  (segment (start 101.6 140.90662) (end 101.6 138.2522) (width 0.25) (layer "B.Cu") (net 9))
   (segment (start 96.139 135.255) (end 97.6375 135.255) (width 0.25) (layer "F.Cu") (net 10))
   (segment (start 93.094 137.13) (end 94.264 137.13) (width 0.25) (layer "F.Cu") (net 10))
@@
         (xy 91.821 124.46)
         (xy 136.017 124.46)
-        (xy 136.017 124.46)
         (xy 136.017 152.527)
         (xy 91.821 152.527)
-        (xy 91.821 152.527)
       )

Commit message: Hardware is almost done
Parts:
- J601: footprint Connector_USB:USB_Micro-B_Amphenol_10118194_Horizontal -> _PCBLIB_EPen:USB_Micro-B_Amphenol_10118194_Horizontal
Routing:
- net Net-(U401-Y4): track 17.4 -> 14.4 mm
- net /BLOCK DIAGRAM/LDO +3V0DC/+3VDC: track 31.9 -> 29.4 mm
Other:
- board text added: "GND ~{MCLR} ~{WP} SCK MOSI MISO ~{CS} GND"
- board text added: "M2.5"
- board text added: "Prj: _HW_EPen Ver: v1.0 Date: 2023/11/28 DES: SiavashTP"
- board text removed: "GND ~{MCLR} ~{WP} SCK MOSI MISO CS GND"
- board text removed: "_HW_EPen v1.0, 2023/11/28 DSN: SiavashTP"

Commit message: Updating file templates and structures...
Parts:
- moved C402 121.5 mm to (171.1, 258.5)
- moved C501 121.5 mm to (155.9, 250.9)
- moved C507 121.5 mm to (158.9, 243.3)
- moved MH801 121.5 mm to (148.3, 257.9)
- moved R302 121.5 mm to (178.8, 244.3)
- moved R404 121.5 mm to (186.4, 247.1)
- moved R702 121.5 mm to (167.3, 258.5)
- moved FD801 121.5 mm to (186.0, 233.9)
- moved J301 121.5 mm to (166.7, 233.1)
- moved MH803 121.5 mm to (192.7, 233.8)
- moved MH804 121.5 mm to (148.3, 233.8)
- moved C301 121.5 mm to (178.1, 242.7)
- moved C302 121.5 mm to (178.1, 241.4)
- moved C303 121.5 mm to (171.0, 236.3)
- moved C502 121.5 mm to (153.4, 254.7)
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Other:
- board text removed: "PCB Layout"
- board text removed: "PRELIMINARY"
