File: Hardware/_Sub_HW_EPen/v1_20231122/Design Folder/_HW_EPen/_HW_EPen.kicad_sch (KiCad schematic)
At the start: 0 parts

Commit message: Working on EPen Schematic
Other:
- added sheet BLOCK DIAGRAM ([02] - BLOCK DIAGRAM.kicad_sch)
- company: (none) -> mend0z0
- title: (none) -> _HW_EPen
Changed lines of the file:
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@@
 (kicad_sch (version 20230121) (generator eeschema)
   (paper "B")
+  (title_block
+    (title "_HW_EPen")
+    (rev "v1.0")
+    (company "mend0z0")
+    (comment 8 "N/A")
+  )
   (polyline (pts (xy 322.58 185.42) (xy 322.58 213.36))
     (stroke (width 0) (type default))
@@
     (effects (font (size 5 5)) (justify left bottom))
   )
+  (sheet (at 50.8 118.11) (size 63.5 6.35) (fields_autoplaced)
+    (stroke (width 0.1524) (type solid))
+    (fill (color 0 0 0 0.0000))
+    (property "Sheetname" "BLOCK DIAGRAM" (at 50.8 117.3984 0)
+      (effects (font (size 1.27 1.27)) (justify left bottom))
+    )
+    (property "Sheetfile" "[02] - BLOCK DIAGRAM.kicad_sch" (at 50.8 125.0446 0)
+      (effects (font (size 1.27 1.27)) (justify left top))
+    )
+    (instances
+      (project "_HW_EPen"
+        (path "/9ee621ae-6984-4881-898c-f5f3c9433407" (page "2"))
+      )
+    )
+  )
   (sheet_instances

Commit message: More progress on EPen Hardware
Other:
- added sheet MECHANICAL PARTS ([08] - MECHANICAL PARTS.kicad_sch)
- note added: "${COMMENT2}"
- note added: "1- Go to View -> Pge Preview Setting 2- Set Parameters based on the following Info COMMENT 1: Project Version COMMENT 2: Document Status COMMENT 3: Doc. Approval Eng. COMMENT 4: BOM Ref. DOC. COMMENT 5: PCB Ref. DOC. COMMENT 6: GBR Ref. DOC. COMMENT 7: ASM Ref. DOC. COMMENT 8: Variant Name COMMENT 9: Revision Description"
- note added: "BLOCK DIAGRAM"
- note added: "FT230X_DRIVER"
- note added: "LDO +3V0DC"
- note added: "MCU"
- note added: "MECHANICAL PARTS"
- note added: "OUTPUT"
- note added: "USB"
- note removed: "1- Go to View -> Pge Preview Setting 2- Set Parameters based on the following Info COMMENT 1: Project Version COMMENT 2: Document Version COMMENT 3: Doc. Approval Eng. COMMENT 4: BOM Ref. DOC. COMMENT 5: PCB Ref. DOC. COMMENT 6: GBR Ref. DOC. COMMENT 7: ASM Ref. DOC. COMMENT 8: Variant Name COMMENT 9: Revision Description"
- note removed: "DRAFT"
Changed lines of the file:
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@@
     (rev "v1.0")
     (company "mend0z0")
+    (comment 1 "v1.0")
+    (comment 2 "PRELIMINARY")
+    (comment 3 "Siavash Taher Parvar")
+    (comment 4 "_BOM_EPen.html")
+    (comment 5 "_HW_EPen.pcb")
+    (comment 6 "_GBR_EPen.zip")
+    (comment 7 "_BOM_EPen.html")
     (comment 8 "N/A")
+    (comment 9 "First Release")
   )
   (polyline (pts (xy 322.58 185.42) (xy 322.58 213.36))
@@
     (effects (font (size 1.8 1.8) bold) (justify left bottom))
   )
+  (text "MECHANICAL PARTS" (at 50.8 200.66 0)
+    (effects (font (size 3.81 3.81)) (justify left bottom))
+  )
   (text "1" (at 29.21 113.03 0)
     (effects (font (size 5 5)) (justify left bottom))
   )
-  (text "1- Go to View -> Pge Preview Setting\n2- Set Parameters based on the following Info\n	COMMENT 1: Project Version\n	COMMENT 2: Document Version\n	COMMENT 3: Doc. Approval Eng.\n	COMMENT 4: BOM Ref. DOC.\n	COMMENT 5: PCB Ref. DOC.\n	COMMENT 6: GBR Ref. DOC.\n	COMMENT 7: ASM Ref. DOC.\n	COMMENT 8: Variant Name\n	COMMENT 9: Revision Description "
+  (text "1- Go to View -> Pge Preview Setting\n2- Set Parameters based on the following Info\n	COMMENT 1: Project Version\n	COMMENT 2: Document Status\n	COMMENT 3: Doc. Approval Eng.\n	COMMENT 4: BOM Ref. DOC.\n	COMMENT 5: PCB Ref. DOC.\n	COMMENT 6: GBR Ref. DOC.\n	COMMENT 7: ASM Ref. DOC.\n	COMMENT 8: Variant Name\n	COMMENT 9: Revision Description "
     (at 262.89 123.19 0)
     (effects (font (size 2.5 2.5)) (justify left bottom))
@@
   (text "Index" (at 50.8 100.33 0)
     (effects (font (size 5 5) italic) (justify left bottom))
+  )
+  (text "USB" (at 50.8 176.53 0)
+    (effects (font (size 6 6)) (justify left bottom))
   )
   (text "DESIGN CONSIDERATION" (at 257.81 182.88 0)
@@
     (effects (font (size 5 5) bold) (justify left bottom))
   )
-  (text "COVER PAGE" (at 52.07 114.3 0)
+  (text "COVER PAGE" (at 50.8 114.3 0)
     (effects (font (size 6 6) italic) (justify left bottom))
   )
@@
     (effects (font (size 6 6) bold italic) (justify left bottom))
   )
+  (text "OUTPUT" (at 50.8 151.13 0)
+    (effects (font (size 6 6)) (justify left bottom))
+  )
   (text "Page" (at 25.4 100.33 0)
     (effects (font (size 5 5) italic) (justify left bottom))
   )
-  (text "DRAFT" (at 99.06 83.82 0)
-    (effects (font (size 7.62 7.62) italic) (justify left bottom))
+  (text "${COMMENT2}" (at 100.33 83.82 0)
+    (effects (font (size 6.35 6.35) (thickness 1.27) bold italic) (justify left bottom))
   )
   (text "12" (at 140.97 124.46 0)
@@
   (text "Page" (at 139.7 100.33 0)
     (effects (font (size 5 5) italic) (justify left bottom))
+  )
+  (text "MCU" (at 50.8 138.43 0)
+    (effects (font (size 6 6)) (justify left bottom))
   )
   (text "13" (at 140.97 137.16 0)
@@
     (effects (font (size 5 5)) (justify left bottom))
   )
-  (text "PWR SEQUENCE" (at 167.64 212.09 0)
+  (text "PWR SEQUENCE" (at 50.8 213.36 0)
     (effects (font (size 4 4)) (justify left bottom))
   )
@@
     (effects (font (size 5 5)) (justify left bottom))
   )
-  (text "REVISION HISTORY" (at 167.64 224.79 0)
+  (text "LDO +3V0DC" (at 50.8 189.23 0)
+    (effects (font (size 6 6)) (justify left bottom))
+  )
+  (text "REVISION HISTORY" (at 50.8 226.06 0)
     (effects (font (size 4 4)) (justify left bottom))
   )
@@
     (effects (font (size 5 5)) (justify left bottom))
   )
+  (text "FT230X_DRIVER" (at 50.8 163.83 0)
+    (effects (font (size 6 6)) (justify left bottom))
+  )
   (text "16" (at 140.97 175.26 0)
     (effects (font (size 5 5)) (justify left bottom))
+  )
+  (text "BLOCK DIAGRAM" (at 50.8 124.46 0)
+    (effects (font (size 3.81 3.81)) (justify left bottom))
   )
   (text "3" (at 29.21 137.16 0)
@@
     (effects (font (size 5 5)) (justify left bottom))
   )
+  (sheet (at 50.8 194.31) (size 63.5 6.35) (fields_autoplaced)
+    (stroke (width 0.1524) (type solid))
+    (fill (color 0 0 0 0.0000))
+    (property "Sheetname" "MECHANICAL PARTS" (at 50.8 193.5984 0)
+      (effects (font (size 1.27 1.27)) (justify left bottom))
+    )
+    (property "Sheetfile" "[08] - MECHANICAL PARTS.kicad_sch" (at 50.8 201.2446 0)
+      (effects (font (size 1.27 1.27)) (justify left top))
+    )
+    (instances
+      (project "_HW_EPen"
+        (path "/9ee621ae-6984-4881-898c-f5f3c9433407" (page "8"))
+      )
+    )
+  )
   (sheet (at 50.8 118.11) (size 63.5 6.35) (fields_autoplaced)

Commit message: _HW_EPen is ready to be worked for layout
Other:
- added sheet PWR SEQUENCE ([09] - PWR SEQUENCE.kicad_sch)
- added sheet REVISION HISTORY ([10] - REVISION HISTORY.kicad_sch)
Changed lines of the file:
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@@
     (company "mend0z0")
     (comment 1 "v1.0")
-    (comment 2 "PRELIMINARY")
+    (comment 2 "CHECKED")
     (comment 3 "Siavash Taher Parvar")
     (comment 4 "_BOM_EPen.html")
@@
     )
   )
+  (sheet (at 50.8 207.01) (size 63.5 6.35) (fields_autoplaced)
+    (stroke (width 0.1524) (type solid))
+    (fill (color 0 0 0 0.0000))
+    (property "Sheetname" "PWR SEQUENCE" (at 50.8 206.2984 0)
+      (effects (font (size 1.27 1.27)) (justify left bottom))
+    )
+    (property "Sheetfile" "[09] - PWR SEQUENCE.kicad_sch" (at 50.8 213.9446 0)
+      (effects (font (size 1.27 1.27)) (justify left top))
+    )
+    (instances
+      (project "_HW_EPen"
+        (path "/9ee621ae-6984-4881-898c-f5f3c9433407" (page "9"))
+      )
+    )
+  )
   (sheet (at 50.8 118.11) (size 63.5 6.35) (fields_autoplaced)
     (stroke (width 0.1524) (type solid))
@@
       )
     )
+  )
+  (sheet (at 50.8 219.71) (size 63.5 6.35) (fields_autoplaced)
+    (stroke (width 0.1524) (type solid))
+    (fill (color 0 0 0 0.0000))
+    (property "Sheetname" "REVISION HISTORY" (at 50.8 218.9984 0)
+      (effects (font (size 1.27 1.27)) (justify left bottom))
+    )
+    (property "Sheetfile" "[10] - REVISION HISTORY.kicad_sch" (at 50.8 226.6446 0)
+      (effects (font (size 1.27 1.27)) (justify left top))
+    )
+    (instances
+      (project "_HW_EPen"
+        (path "/9ee621ae-6984-4881-898c-f5f3c9433407" (page "10"))
+      )
+    )

Commit message: Updating Hardware File structures
Other:
- note added: "21"
- note added: "22"
- note added: "23"
- note added: "24"
- note added: "25"
- note added: "26"
- note added: "27"
- note added: "28"
- note added: "29"
- note added: "30"
- note added: "3D Preview BOTTOM"
- note added: "3D Preview TOP"
- note added: "Board Statistics Stackup Info"
- note added: "SHOULD BE ADDED AFTER RELEASE"
