File: Hardware/_Sub_HW_EPaper/v1_20231122/Design Folder/_HW_EPaper/[03] - MCU.kicad_sch (KiCad schematic)
At the start: 7 parts, among them J301 HDR_4POS_VERT, U301 PIC16F15223_8BIT

Commit message: Latest update
Parts:
- C301, C303: symbol _SCHLIB_EPen:CAP_100nF_50V_X7R_C0402 -> _SCHLIB_Epaper:CAP_100nF_50V_X7R_C0402
- C302: symbol _SCHLIB_EPen:CAP_1uF_10V_X7R_C0402 -> _SCHLIB_Epaper:CAP_1uF_10V_X7R_C0402
- J301: symbol _SCHLIB_EPen:CONN_HEADER_4POS_1ROW_VERT_2.54mm -> _SCHLIB_Epaper:CONN_HEADER_4POS_1ROW_VERT_2.54mm
- R301: symbol _SCHLIB_EPen:RES_10kR_1/16W_1%_R0402 -> _SCHLIB_Epaper:RES_10kR_1/16W_1%_R0402
- R302: symbol _SCHLIB_EPen:RES_1R_1/4W_1%_R0805 -> _SCHLIB_Epaper:RES_1R_1/4W_1%_R0805
- U301: symbol _SCHLIB_EPen:MCU_PIC16F15223-E/SL_8BIT_14-SOIC -> _SCHLIB_Epaper:MCU_PIC16F15223-E/SL_8BIT_14-SOIC
Connections:
- no-connect marks 0 -> 1
Other:
- moved on the sheet: C301
Changed lines of the file:
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@@
     (company "Mend0z0")
     (comment 1 "v1.0")
-    (comment 2 "DRAFT")
+    (comment 2 "PRELIMINARY")
   )
   (junction (at 135.89 128.27) (diameter 0) (color 0 0 0 0)
   )
-  (junction (at 154.94 146.05) (diameter 0) (color 0 0 0 0)
-  )
-  (junction (at 154.94 128.27) (diameter 0) (color 0 0 0 0)
+  (junction (at 156.21 146.05) (diameter 0) (color 0 0 0 0)
   )
   (junction (at 135.89 146.05) (diameter 0) (color 0 0 0 0)
@@
   (junction (at 135.89 104.14) (diameter 0) (color 0 0 0 0)
   )
+  (junction (at 156.21 128.27) (diameter 0) (color 0 0 0 0)
+  )
+  (no_connect (at 215.9 125.73))
   (wire (pts (xy 135.89 118.11) (xy 135.89 119.38))
     (stroke (width 0) (type default))
   )
-  (wire (pts (xy 154.94 128.27) (xy 154.94 130.81))
+  (wire (pts (xy 156.21 128.27) (xy 156.21 130.81))
     (stroke (width 0) (type default))
   )
@@
     (stroke (width 0) (type default))
   )
-  (wire (pts (xy 175.26 146.05) (xy 154.94 146.05))
-    (stroke (width 0) (type default))
-  )
-  (wire (pts (xy 135.89 146.05) (xy 154.94 146.05))
+  (wire (pts (xy 175.26 146.05) (xy 156.21 146.05))
     (stroke (width 0) (type default))
   )
@@
     (stroke (width 0) (type default))
   )
+  (wire (pts (xy 135.89 128.27) (xy 156.21 128.27))
+    (stroke (width 0) (type default))
+  )
   (wire (pts (xy 135.89 146.05) (xy 135.89 147.32))
     (stroke (width 0) (type default))
@@
     (stroke (width 0) (type default))
   )
-  (wire (pts (xy 231.14 125.73) (xy 213.36 125.73))
+  (wire (pts (xy 215.9 125.73) (xy 213.36 125.73))
     (stroke (width 0) (type default))
   )
@@
     (stroke (width 0) (type default))
   )
-  (wire (pts (xy 135.89 128.27) (xy 154.94 128.27))
-    (stroke (width 0) (type default))
-  )
   (wire (pts (xy 231.14 130.81) (xy 213.36 130.81))
     (stroke (width 0) (type default))
@@
     (stroke (width 0) (type default))
   )
-  (wire (pts (xy 177.8 128.27) (xy 154.94 128.27))
+  (wire (pts (xy 177.8 128.27) (xy 156.21 128.27))
     (stroke (width 0) (type default))
   )
@@
     (stroke (width 0) (type default))
   )
+  (wire (pts (xy 135.89 146.05) (xy 156.21 146.05))
+    (stroke (width 0) (type default))
+  )
   (polyline (pts (xy 130.81 130.81) (xy 119.38 130.81))
     (stroke (width 0) (type default))
   )
-  (wire (pts (xy 154.94 146.05) (xy 154.94 143.51))
+  (wire (pts (xy 156.21 146.05) (xy 156.21 143.51))
     (stroke (width 0) (type default))
   )
@@
     (fill (type none))
   )
-  (circle (center 154.94 128.27) (radius 1.27)
+  (circle (center 156.21 128.27) (radius 1.27)
     (stroke (width 0) (type default))
     (fill (type none))
@@
     (effects (font (size 1.27 1.27)) (justify left bottom))
   )
-  (text "HPF2" (at 156.21 127 0)
+  (text "HPF2" (at 157.48 127 0)
     (effects (font (size 1.27 1.27)) (justify left bottom))
   )
@@
     (effects (font (size 1.27 1.27)) (justify right))
   )
-  (symbol (lib_id "_SCHLIB_EPen:MCU_PIC16F15223-E/SL_8BIT_14-SOIC") (at 182.88 101.6 0) (unit 1)
+  (symbol (lib_id "_SCHLIB_Epaper:MCU_PIC16F15223-E/SL_8BIT_14-SOIC") (at 182.88 101.6 0) (unit 1)
     (in_bom yes) (on_board yes) (dnp no) (fields_autoplaced)
     (property "Reference" "U301" (at 195.58 88.9 0)
@@
     )
   )
-  (symbol (lib_id "_SCHLIB_EPen:CAP_1uF_10V_X7R_C0402") (at 135.89 130.81 270) (unit 1)
+  (symbol (lib_id "_SCHLIB_Epaper:CAP_1uF_10V_X7R_C0402") (at 135.89 130.81 270) (unit 1)
     (in_bom yes) (on_board yes) (dnp no) (fields_autoplaced)
     (property "Reference" "C302" (at 138.43 132.08 90)
@@
     )
   )
-  (symbol (lib_id "_SCHLIB_EPen:CAP_100nF_50V_X7R_C0402") (at 154.94 130.81 270) (unit 1)
-    (in_bom yes) (on_board yes) (dnp no) (fields_autoplaced)
-    (property "Reference" "C301" (at 157.48 132.08 90)
-      (effects (font (size 1.27 1.27)) (justify left))
-    )
-    (property "Value" "100nF_50V" (at 157.48 134.62 90)
-      (effects (font (size 1.27 1.27)) (justify left))
-    )
-    (property "Footprint" "Capacitor_SMD:C_0402_1005Metric" (at 171.45 133.35 0)
-      (effects (font (size 1.27 1.27)) (justify left) hide)
-    )
-    (property "Datasheet" "https://search.murata.co.jp/Ceramy/image/img/A01X/G101/ENG/GRM155R71H104KE14-01.pdf" (at 163.83 133.35 0)
-      (effects (font (size 1.27 1.27)) (justify left) hide)
-    )
-    (property "Description" "0.1 µF ±10% 50V Ceramic Capacitor X7R 0402 (1005 Metric)" (at 168.91 133.35 0)
-      (effects (font (size 1.27 1.27)) (justify left) hide)
-    )
-    (property "Part Number" "GRM155R71H104KE14J" (at 173.99 133.35 0)
-      (effects (font (size 1.27 1.27)) (justify left) hide)
-    )
-    (property "Link" "https://www.digikey.ca/en/products/detail/murata-electronics/GRM155R71H104KE14J/4905180" (at 166.37 133.35 0)
-      (effects (font (size 1.27 1.27)) (justify left) hide)
-    )
-    (property "Package" "C0402" (at 157.48 137.16 90)
-      (effects (font (size 1.27 1.27)) (justify left))
-    )
-    (property "SCH CHECK" "SCH (CHECKED)" (at 157.48 139.7 90)
-      (effects (font (size 1.27 1.27)) (justify left))
-    )
-    (property "PCB CHECK" "PCB (N/A)" (at 157.48 142.24 90)
+  (symbol (lib_id "_SCHLIB_Epaper:CAP_100nF_50V_X7R_C0402") (at 156.21 130.81 270) (unit 1)
+    (in_bom yes) (on_board yes) (dnp no) (fields_autoplaced)
+    (property "Reference" "C301" (at 158.75 132.08 90)
+      (effects (font (size 1.27 1.27)) (justify left))
+    )
+    (property "Value" "100nF_50V" (at 158.75 134.62 90)
+      (effects (font (size 1.27 1.27)) (justify left))
+    )
+    (property "Footprint" "Capacitor_SMD:C_0402_1005Metric" (at 172.72 133.35 0)
+      (effects (font (size 1.27 1.27)) (justify left) hide)
+    )
+    (property "Datasheet" "https://search.murata.co.jp/Ceramy/image/img/A01X/G101/ENG/GRM155R71H104KE14-01.pdf" (at 165.1 133.35 0)
+      (effects (font (size 1.27 1.27)) (justify left) hide)
+    )
+    (property "Description" "0.1 µF ±10% 50V Ceramic Capacitor X7R 0402 (1005 Metric)" (at 170.18 133.35 0)
+      (effects (font (size 1.27 1.27)) (justify left) hide)
+    )
+    (property "Part Number" "GRM155R71H104KE14J" (at 175.26 133.35 0)
+      (effects (font (size 1.27 1.27)) (justify left) hide)
+    )
+    (property "Link" "https://www.digikey.ca/en/products/detail/murata-electronics/GRM155R71H104KE14J/4905180" (at 167.64 133.35 0)
+      (effects (font (size 1.27 1.27)) (justify left) hide)
+    )
+    (property "Package" "C0402" (at 158.75 137.16 90)
+      (effects (font (size 1.27 1.27)) (justify left))
+    )
+    (property "SCH CHECK" "SCH (CHECKED)" (at 158.75 139.7 90)
+      (effects (font (size 1.27 1.27)) (justify left))
+    )
+    (property "PCB CHECK" "PCB (N/A)" (at 158.75 142.24 90)
       (effects (font (size 1.27 1.27)) (justify left))
     )
@@
     )
   )
-  (symbol (lib_id "_SCHLIB_EPen:RES_1R_1/4W_1%_R0805") (at 91.44 128.27 0) (unit 1)
+  (symbol (lib_id "_SCHLIB_Epaper:RES_1R_1/4W_1%_R0805") (at 91.44 128.27 0) (unit 1)
     (in_bom yes) (on_board yes) (dnp no)
     (property "Reference" "R302" (at 106.68 127 0)
@@
       (effects (font (size 1.27 1.27)) (justify left) hide)
     )
-    (property "Package" "R0805" (at 88.9 129.54 0)
-      (effects (font (size 1.27 1.27)))
-    )
-    (property "SCH CHECK" "SCH (CHECKED)" (at 111.76 129.54 0)
-      (effects (font (size 1.27 1.27)))
-    )
-    (property "PCB CHECK" "PCB (N/A)" (at 109.22 132.08 0)
-      (effects (font (size 1.27 1.27)))
+    (property "Package" "R0805" (at 85.09 129.54 0)
+      (effects (font (size 1.27 1.27)) (justify left))
+    )
+    (property "SCH CHECK" "SCH (CHECKED)" (at 104.14 129.54 0)
+      (effects (font (size 1.27 1.27)) (justify left))
+    )
+    (property "PCB CHECK" "PCB (N/A)" (at 104.14 132.08 0)
+      (effects (font (size 1.27 1.27)) (justify left))
     )
     (pin "1")
@@
     )
   )
-  (symbol (lib_id "_SCHLIB_EPen:CONN_HEADER_4POS_1ROW_VERT_2.54mm") (at 195.58 157.48 0) (unit 1)
+  (symbol (lib_id "_SCHLIB_Epaper:CONN_HEADER_4POS_1ROW_VERT_2.54mm") (at 195.58 157.48 0) (unit 1)
     (in_bom yes) (on_board yes) (dnp no) (fields_autoplaced)
     (property "Reference" "J301" (at 201.93 158.75 0)
@@
     )
   )
-  (symbol (lib_id "_SCHLIB_EPen:CAP_100nF_50V_X7R_C0402") (at 135.89 105.41 270) (unit 1)
+  (symbol (lib_id "_SCHLIB_Epaper:CAP_100nF_50V_X7R_C0402") (at 135.89 105.41 270) (unit 1)
     (in_bom yes) (on_board yes) (dnp no) (fields_autoplaced)
     (property "Reference" "C303" (at 138.43 106.68 90)
@@
     )
   )
-  (symbol (lib_id "_SCHLIB_EPen:RES_10kR_1/16W_1%_R0402") (at 135.89 90.17 270) (unit 1)
+  (symbol (lib_id "_SCHLIB_Epaper:RES_10kR_1/16W_1%_R0402") (at 135.89 90.17 270) (unit 1)
     (in_bom yes) (on_board yes) (dnp no) (fields_autoplaced)
     (property "Reference" "R301" (at 138.43 91.44 90)
