File: Hardware/_Sub_HW_EPaper/v1_20231122/Design Folder/_HW_EPaper/[06] - SIPO.kicad_sch (KiCad schematic)
At the start: 3 parts, among them U601 74VHC164FT

Commit message: Working on epaper hardware
Connections:
- net DISPLAY_D/C: now also U601.11 (QF); no longer U601.5 (QC)
- net DISPLAY_PWR: now also U601.10 (QE); no longer U601.6 (QD)
- net DISPLAY_~{CS}: now also U601.13 (QH); no longer U601.3 (QA)
- net DISPLAY_~{RST}: now also U601.12 (QG); no longer U601.4 (QB)
- net LED_1: now also U601.4 (QB); no longer U601.12 (QG)
- net LED_2: now also U601.3 (QA); no longer U601.13 (QH)
- net SF_HOLD: now also U601.5 (QC); no longer U601.11 (QF)
- net SF_~{CS}: now also U601.6 (QD); no longer U601.10 (QE)
Changed lines of the file:
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@@
     (company "Mend0z0")
     (comment 1 "v1.0")
-    (comment 2 "PRELIMINARY")
+    (comment 2 "CHECKED")
   )
   (junction (at 160.02 116.84) (diameter 0) (color 0 0 0 0)
@@
     (effects (font (size 1.27 1.27)) (justify left bottom))
   )
-  (hierarchical_label "SF_~{CS}" (shape output) (at 215.9 114.3 0) (fields_autoplaced)
-    (effects (font (size 1.27 1.27)) (justify left))
-  )
   (hierarchical_label "VIN" (shape input) (at 152.4 116.84 180) (fields_autoplaced)
     (effects (font (size 1.27 1.27)) (justify right))
   )
-  (hierarchical_label "LED_2" (shape output) (at 215.9 121.92 0) (fields_autoplaced)
+  (hierarchical_label "SF_HOLD" (shape output) (at 215.9 109.22 0) (fields_autoplaced)
     (effects (font (size 1.27 1.27)) (justify left))
   )
@@
     (effects (font (size 1.27 1.27)) (justify right))
   )
+  (hierarchical_label "DISPLAY_~{CS}" (shape output) (at 215.9 121.92 0) (fields_autoplaced)
+    (effects (font (size 1.27 1.27)) (justify left))
+  )
+  (hierarchical_label "LED_1" (shape output) (at 215.9 106.68 0) (fields_autoplaced)
+    (effects (font (size 1.27 1.27)) (justify left))
+  )
   (hierarchical_label "74VHC164_DAT" (shape input) (at 167.64 107.95 180) (fields_autoplaced)
     (effects (font (size 1.27 1.27)) (justify right))
   )
-  (hierarchical_label "DISPLAY_~{CS}" (shape output) (at 215.9 104.14 0) (fields_autoplaced)
-    (effects (font (size 1.27 1.27)) (justify left))
-  )
-  (hierarchical_label "DISPLAY_~{RST}" (shape output) (at 215.9 106.68 0) (fields_autoplaced)
-    (effects (font (size 1.27 1.27)) (justify left))
-  )
-  (hierarchical_label "DISPLAY_D{slash}C" (shape output) (at 215.9 109.22 0) (fields_autoplaced)
+  (hierarchical_label "DISPLAY_D{slash}C" (shape output) (at 215.9 116.84 0) (fields_autoplaced)
     (effects (font (size 1.27 1.27)) (justify left))
   )
@@
     (effects (font (size 1.27 1.27)) (justify right))
   )
-  (hierarchical_label "SF_HOLD" (shape output) (at 215.9 116.84 0) (fields_autoplaced)
+  (hierarchical_label "DISPLAY_PWR" (shape output) (at 215.9 114.3 0) (fields_autoplaced)
     (effects (font (size 1.27 1.27)) (justify left))
   )
-  (hierarchical_label "DISPLAY_PWR" (shape output) (at 215.9 111.76 0) (fields_autoplaced)
+  (hierarchical_label "DISPLAY_~{RST}" (shape output) (at 215.9 119.38 0) (fields_autoplaced)
     (effects (font (size 1.27 1.27)) (justify left))
   )
-  (hierarchical_label "LED_1" (shape output) (at 215.9 119.38 0) (fields_autoplaced)
+  (hierarchical_label "SF_~{CS}" (shape output) (at 215.9 111.76 0) (fields_autoplaced)
     (effects (font (size 1.27 1.27)) (justify left))
   )
+  (hierarchical_label "LED_2" (shape output) (at 215.9 104.14 0) (fields_autoplaced)
+    (effects (font (size 1.27 1.27)) (justify left))
+  )

Commit message: Updating file templates and structures...
Parts:
- C601: Manufacturer (none) -> Murata Electronics; Part Number GRM155Z71A105KE01D -> (none); Part Number (Manufacturer) (none) -> GRM155Z71A105KE01D; Part Number (Vendor) (none) -> 490-GRM155Z71A105KE01DTR-ND; Vendor (none) -> Digikey
- R601: Manufacturer (none) -> Bourns Inc.; Part Number CR0402-FX-1002GLF -> (none); Part Number (Manufacturer) (none) -> CR0402-FX-1002GLF; Part Number (Vendor) (none) -> CR0402-FX-1002GLFTR-ND; Vendor (none) -> Digikey
- U601: Manufacturer (none) -> Toshiba Semiconductor and Storage; Part Number 74VHC164FT -> (none); Part Number (Manufacturer) (none) -> 74VHC164FT; Part Number (Vendor) (none) -> 264-74VHC164FTTR-ND; Vendor (none) -> Digikey
Other:
- moved on the sheet: C601, R601, U601
