File: Hardware/_Sub_HW_EPaper/v1_20231122/Design Folder/_HW_EPaper/[05] - INPUT CIRCUIT.kicad_sch (KiCad schematic)
At the start: 0 parts

Commit message: Working on E-Paper schematic
Parts:
- added C501: 1uF_10V_X7R, Capacitor_SMD:C_0402_1005Metric, symbol _SCHLIB_Epaper:CAP_1uF_10V_X7R_C0402
- added D501, D502, D503, D504, D505: TVS_6.5V_3A, _PCBLIB_Epaper:CR_7PCT_L3F_TOS, symbol _SCHLIB_Epaper:TVS_5V(MAX)_6.5(Vbr-min)_3A(8/20us)_SOD882
- added J501: RECEPT_8POS_RA, Connector_PinSocket_2.54mm:PinSocket_1x08_P2.54mm_Horizontal, symbol _SCHLIB_Epaper:CONN_RECEPT_8POS_1RAW_RA_2.54mm
- added R501, R502, R503, R504, R505, R506, R507: 10kR_1/16W_1%, Resistor_SMD:R_0402_1005Metric, symbol _SCHLIB_Epaper:RES_10kR_1/16W_1%_R0402
- added R508, R509, R510, R511: 27R_1/16W_1%, Resistor_SMD:R_0402_1005Metric, symbol _SCHLIB_Epaper:RES_27R_1/16W_1%_R0402
- added U501: SN74HCS32PWR, Package_SO:TSSOP-14_4.4x5mm_P0.65mm, symbol _SCHLIB_Epaper:IC_OR GATE_SN74HCS32PWR_4CH_2-INP_14-TSSOP
Connections:
- new net: D502.1, R503.1, R509.2, U501.10 (3B)
- new net: D501.1, R505.1, R508.2, U501.5 (2B)
- new net EXTERNAL_EEPROM_~{WP}: J501.6, R510.1
- new net EXTERNAL_MCU_~{MCLR}: J501.7, R511.1
- new net EXTERNAL_SPI_MOSI: J501.4, R509.1
- new net EXTERNAL_SPI_SCK: J501.5, R508.1
- new net EXTERNAL_SPI_~{CS}: J501.2, R502.2, U501.2 (1B)
- new net GND: C501.2, D501.2, D502.2, D503.2, D504.2, D505.2, J501.1, J501.8, R503.2, R504.2, R505.2, R506.2, R507.2, U501.7 (GND)
- new net MCU_SPI_CLK: R506.1, U501.4 (2A)
- new net MCU_SPI_MOSI: R504.1, U501.9 (3A)
- new net MCU_SPI_~{CS}: R501.2, U501.1 (1A)
- new net MCU_~{RESET}: D505.1, R511.2
- new net SF_CLK: U501.6 (2Y)
- new net SF_DI: U501.8 (3Y)
- new net SF_DO: D503.1, R507.1, U501.12 (4A), U501.13 (4B)
- new net SF_~{CS}: U501.3 (1Y)
- new net SF_~{WP}: D504.1, R510.2
- new net SPI_MISO: J501.3, U501.11 (4Y)
- new net VIN: C501.1, R501.1, R502.1, U501.14 (VCC)
Other:
- note added: "LAYOUT NOTE:"

Commit message: Latest update
Parts:
- J501: Package Through Hole (RA) -> Through Hole (2.54mm)
Changed lines of the file:
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@@
     (company "Mend0z0")
     (comment 1 "v1.0")
-    (comment 2 "DRAFT")
+    (comment 2 "PRELIMINARY")
   )
   (junction (at 219.71 91.44) (diameter 0) (color 0 0 0 0)
@@
       (effects (font (size 1.27 1.27)) (justify left) hide)
     )
-    (property "Package" "Through Hole (RA)" (at 41.91 157.48 0)
+    (property "Package" "Through Hole (2.54mm)" (at 41.91 157.48 0)
       (effects (font (size 1.27 1.27)))
     )

Commit message: Working on epaper hardware
Parts:
- removed D503: TVS_6.5V_3A, _PCBLIB_Epaper:CR_7PCT_L3F_TOS, symbol _SCHLIB_Epaper:TVS_5V(MAX)_6.5(Vbr-min)_3A(8/20us)_SOD882
- renumbered D504 to D503, D505 to D504, R502 to R501, R501 to R502, R508 to R503, R509 to R504, R503 to R508, R504 to R509

Commit message: Hardware is almost done
Parts:
- removed J501: RECEPT_8POS_RA, Connector_PinSocket_2.54mm:PinSocket_1x08_P2.54mm_Horizontal, symbol _SCHLIB_Epaper:CONN_RECEPT_8POS_1RAW_RA_2.54mm
- added J501: HDR_8POS_RA, Connector_PinHeader_2.54mm:PinHeader_1x08_P2.54mm_Horizontal, symbol _SCHLIB_Epaper:CONN_HEADER_8POS_1RAW_RA_2.54mm
Connections:
- net EXTERNAL_EEPROM_~{WP}: now also J501.3
- net EXTERNAL_MCU_~{MCLR}: now also J501.2
- net EXTERNAL_SPI_MOSI: now also J501.5
- net EXTERNAL_SPI_SCK: now also J501.4
- net EXTERNAL_SPI_~{CS}: now also J501.7
- net GND: now also J501.1, J501.8
- net SPI_MISO: now also J501.6
Changed lines of the file:
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@@
-    )
-  )
-  (symbol (lib_id "_SCHLIB_Epaper:CONN_RECEPT_8POS_1RAW_RA_2.54mm") (at 44.45 187.96 180) (unit 1)
-    (in_bom yes) (on_board yes) (dnp no) (fields_autoplaced)
-    (property "Reference" "J501" (at 41.91 152.4 0)
-      (effects (font (size 1.27 1.27)))
-    )
-    (property "Value" "RECEPT_8POS_RA" (at 41.91 154.94 0)
-      (effects (font (size 1.27 1.27)))
-    )
-    (property "Footprint" "Connector_PinSocket_2.54mm:PinSocket_1x08_P2.54mm_Horizontal" (at 41.91 204.47 0)
-      (effects (font (size 1.27 1.27)) (justify left) hide)
-    )
-    (property "Datasheet" "http://suddendocs.samtec.com/catalog_english/ssq_th.pdf" (at 41.91 196.85 0)
-      (effects (font (size 1.27 1.27)) (justify left) hide)
-    )
-    (property "Description" "8 Position Receptacle Connector 0.100\" (2.54mm) Through Hole, Right Angle Tin" (at 41.91 201.93 0)
-      (effects (font (size 1.27 1.27)) (justify left) hide)
-    )
-    (property "Part Number" "SSQ-108-02-T-S-RA" (at 41.91 207.01 0)
-      (effects (font (size 1.27 1.27)) (justify left) hide)
-    )
-    (property "Link" "https://www.digikey.ca/en/products/detail/samtec-inc/SSQ-108-02-T-S-RA/1111404" (at 41.91 199.39 0)
-      (effects (font (size 1.27 1.27)) (justify left) hide)
-    )
-    (property "Package" "Through Hole (2.54mm)" (at 41.91 157.48 0)
-      (effects (font (size 1.27 1.27)))
-    )
-    (property "SCH CHECK" "SCH (CHECKED)" (at 41.91 160.02 0)
-      (effects (font (size 1.27 1.27)))
-    )
-    (property "PCB CHECK" "PCB (N/A)" (at 41.91 162.56 0)
-      (effects (font (size 1.27 1.27)))
-    )
-    (pin "1")
-    (pin "6")
-    (pin "2")
-    (pin "4")
-    (pin "7")
-    (pin "8")
-    (pin "3")
-    (pin "5")
-    (instances
-      (project "_HW_EPaper"
-        (path "/adfaa0ae-c952-44c7-bc24-1bfe8f9a84a3/4e346fc8-747a-4f3e-83e0-81c9211edb38/6221c7ba-76d0-4b5a-99b8-b96cf2af5bf0"
-          (reference "J501") (unit 1)
-        )
-      )
     )
   )
@@
         )
       )
+    )
+  )
+  (symbol (lib_id "_SCHLIB_Epaper:CONN_HEADER_8POS_1RAW_RA_2.54mm") (at 44.45 165.1 0) (mirror y) (unit 1)
+    (in_bom yes) (on_board yes) (dnp no) (fields_autoplaced)
+    (property "Reference" "J501" (at 41.91 152.4 0)
+      (effects (font (size 1.27 1.27)))
+    )
+    (property "Value" "HDR_8POS_RA" (at 41.91 154.94 0)
+      (effects (font (size 1.27 1.27)))
+    )
+    (property "Footprint" "Connector_PinHeader_2.54mm:PinHeader_1x08_P2.54mm_Horizontal" (at 41.91 148.59 0)
+      (effects (font (size 1.27 1.27)) (justify left) hide)
+    )
+    (property "Datasheet" "https://app.adam-tech.com/products/download/data_sheet/201281/ph1rb-xx-ua-data-sheet.pdf" (at 41.91 156.21 0)
+      (effects (font (size 1.27 1.27)) (justify left) hide)
+    )
+    (property "Description" "Connector Header Through Hole, Right Angle 8 position 0.100\" (2.54mm)" (at 41.91 151.13 0)
+      (effects (font (size 1.27 1.27)) (justify left) hide)
+    )
+    (property "Part Number" "PH1RB-08-UA" (at 41.91 146.05 0)
+      (effects (font (size 1.27 1.27)) (justify left) hide)
+    )
+    (property "Link" "https://www.digikey.ca/en/products/detail/adam-tech/PH1RB-08-UA/9831008" (at 41.91 153.67 0)
+      (effects (font (size 1.27 1.27)) (justify left) hide)
+    )
+    (property "Package" "Through Hole (2.54mm)" (at 41.91 157.48 0)
+      (effects (font (size 1.27 1.27)))
+    )
+    (property "SCH CHECK" "SCH (CHECKED)" (at 41.91 160.02 0)
+      (effects (font (size 1.27 1.27)))
+    )
+    (property "PCB CHECK" "PCB (N/A)" (at 41.91 162.56 0)
+      (effects (font (size 1.27 1.27)))
+    )
+    (pin "7")
+    (pin "5")
+    (pin "3")
+    (pin "8")
+    (pin "4")
+    (pin "6")
+    (pin "1")
+    (pin "2")
+    (instances
+      (project "_HW_EPaper"
+        (path "/adfaa0ae-c952-44c7-bc24-1bfe8f9a84a3/4e346fc8-747a-4f3e-83e0-81c9211edb38/6221c7ba-76d0-4b5a-99b8-b96cf2af5bf0"
+          (reference "J501") (unit 1)
+        )
+      )

Commit message: Updating file templates and structures...
Parts:
- C501: Manufacturer (none) -> Murata Electronics; Part Number GRM155Z71A105KE01D -> (none); Part Number (Manufacturer) (none) -> GRM155Z71A105KE01D; Part Number (Vendor) (none) -> 490-GRM155Z71A105KE01DTR-ND; Vendor (none) -> Digikey
- D501, D502, D503, D504: Manufacturer (none) -> Good-Ark Semiconductor; Part Number GSEWT5B003 -> (none); Part Number (Manufacturer) (none) -> GSEWT5B003; Part Number (Vendor) (none) -> 4786-GSEWT5B003TR-ND; Vendor (none) -> Digikey
- J501: Manufacturer (none) -> Adam Tech; Part Number PH1RB-08-UA -> (none); Part Number (Manufacturer) (none) -> PH1RB-08-UA; Part Number (Vendor) (none) -> 2057-PH1RB-08-UA-ND; Vendor (none) -> Digikey
- R501, R502, R505, R506, R507, R508, R509: Manufacturer (none) -> Bourns Inc.; Part Number CR0402-FX-1002GLF -> (none); Part Number (Manufacturer) (none) -> CR0402-FX-1002GLF; Part Number (Vendor) (none) -> CR0402-FX-1002GLFTR-ND; Vendor (none) -> Digikey
- R503, R504, R510, R511: Manufacturer (none) -> Bourns Inc.; Part Number CR0402-FX-27R0GLF -> (none); Part Number (Manufacturer) (none) -> CR0402-FX-27R0GLF; Part Number (Vendor) (none) -> CR0402-FX-27R0GLFTR-ND; Vendor (none) -> Digikey
- U501: Manufacturer (none) -> Texas Instruments; Part Number SN74HCS32PWR -> (none); Part Number (Manufacturer) (none) -> SN74HCS32PWR; Part Number (Vendor) (none) -> 296-SN74HCS32PWRTR-ND; Vendor (none) -> Digikey
Other:
- moved on the sheet: C501, D501, D502, D503, D504, J501, R501, R502, R503, R504, R505, R506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
