File: Hardware/_Sub_HW_EPaper/v1_20231122/Design Folder/_HW_EPaper/[09] - TEMP SENSOR.kicad_sch (KiCad schematic)
At the start: 3 parts, among them U901 MCP9700T-E/TT

Commit message: Hardware is almost done
Parts:
- U901: footprint Package_TO_SOT_SMD:SOT-23-3 -> Package_TO_SOT_SMD:SOT-23; PCB CHECK PCB (N/A) -> PCB (CHECKED); SCH CHECK SCH (N/A) -> SCH (CHECKED)
Changed lines of the file:
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@@
       (effects (font (size 1.27 1.27)))
     )
-    (property "Footprint" "Package_TO_SOT_SMD:SOT-23-3" (at 191.77 97.79 0)
+    (property "Footprint" "Package_TO_SOT_SMD:SOT-23" (at 191.77 97.79 0)
       (effects (font (size 1.27 1.27)) (justify left) hide)
     )
@@
       (effects (font (size 1.27 1.27)))
     )
-    (property "SCH CHECK" "SCH (N/A)" (at 203.2 109.22 0)
+    (property "SCH CHECK" "SCH (CHECKED)" (at 203.2 109.22 0)
       (effects (font (size 1.27 1.27)))
     )
-    (property "PCB CHECK" "PCB (N/A)" (at 203.2 111.76 0)
+    (property "PCB CHECK" "PCB (CHECKED)" (at 203.2 111.76 0)
       (effects (font (size 1.27 1.27)))
     )

Commit message: Updating file templates and structures...
Parts:
- C901: Manufacturer (none) -> Murata Electronics; Part Number GRM155Z71A105KE01D -> (none); Part Number (Manufacturer) (none) -> GRM155Z71A105KE01D; Part Number (Vendor) (none) -> 490-GRM155Z71A105KE01DTR-ND; Vendor (none) -> Digikey
- R901: Manufacturer (none) -> Bourns Inc.; Part Number CR0402-FX-1002GLF -> (none); Part Number (Manufacturer) (none) -> CR0402-FX-1002GLF; Part Number (Vendor) (none) -> CR0402-FX-1002GLFTR-ND; Vendor (none) -> Digikey
- U901: Manufacturer (none) -> Microchip Technology; Part Number MCP9700T-E/TT -> (none); Part Number (Manufacturer) (none) -> MCP9700T-E/TT; Part Number (Vendor) (none) -> MCP9700T-E/TTTR-ND; Vendor (none) -> Digikey
Other:
- moved on the sheet: C901, R901, U901
