File: Hardware/_Sub_HW_EPaper/v1_20231122/Design Folder/_HW_EPaper/[14] - REVISION HISTORY.kicad_sch (KiCad schematic)
At the start: 0 parts

Commit message: Updating Hardware File structures
Other:
- company: mend0z0 -> Mend0z0
- title: _HW_EPen -> _HW_EPaper
Changed lines of the file:
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@@
   (paper "C")
   (title_block
-    (title "_HW_EPen")
-    (date "2023/11/28")
+    (title "_HW_EPaper")
+    (date "2023-12-18")
     (rev "v1.0")
-    (company "mend0z0")
+    (company "Mend0z0")
     (comment 1 "v1.0")
     (comment 2 "CHECKED")
     (comment 3 "Siavash Taher Parvar")
-    (comment 4 "_BOM_EPen.csv")
-    (comment 5 "_HW_EPen.kicad_pcb")
-    (comment 6 "_GBR_EPen.zip")
-    (comment 7 "_BOM_EPen.html")
+    (comment 4 "_BOM_EPaper.csv")
+    (comment 5 "_HW_EPaper.kicad_pcb")
+    (comment 6 "_GBR_EPaper.zip")
+    (comment 7 "_ASM_EPaper.html")
     (comment 8 "N/A")
     (comment 9 "First Release")
