File: Hardware/_Sub_HW_EPaper/v1_20231122/Design Folder/_HW_EPaper/_HW_EPaper.kicad_sch (KiCad schematic)
At the start: 0 parts

Commit message: Working on EPaper Schematic
Other:
- added sheet BLOCK DIAGRAM ([02] - BLOCK DIAGRAM.kicad_sch)
- note added: "1- Go to View -> Pge Preview Setting 2- Set Parameters based on the following Info COMMENT 1: Project Version COMMENT 2: Document Status COMMENT 3: Doc. Approval Eng. COMMENT 4: BOM Ref. DOC. COMMENT 5: PCB Ref. DOC. COMMENT 6: GBR Ref. DOC. COMMENT 7: ASM Ref. DOC. COMMENT 8: Variant Name COMMENT 9: Revision Description"
- note removed: "1- Go to View -> Pge Preview Setting 2- Set Parameters based on the following Info COMMENT 1: Project Version COMMENT 2: Document Version COMMENT 3: Doc. Approval Eng. COMMENT 4: BOM Ref. DOC. COMMENT 5: PCB Ref. DOC. COMMENT 6: GBR Ref. DOC. COMMENT 7: ASM Ref. DOC. COMMENT 8: Variant Name COMMENT 9: Revision Description"
- company: (none) -> Mend0z0
- title: (none) -> _HW_EPaper

Commit message: EPaper schematic is almost done...
Other:
- added sheet MECHANICAL PARTS ([12] - MECHANICAL PARTS.kicad_sch)
Changed lines of the file:
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@@
+    )
+  )
+  (sheet (at 50.8 194.31) (size 63.5 6.35) (fields_autoplaced)
+    (stroke (width 0.1524) (type solid))
+    (fill (color 0 0 0 0.0000))
+    (property "Sheetname" "MECHANICAL PARTS" (at 50.8 193.5984 0)
+      (effects (font (size 1.27 1.27)) (justify left bottom))
+    )
+    (property "Sheetfile" "[12] - MECHANICAL PARTS.kicad_sch" (at 50.8 201.2446 0)
+      (effects (font (size 1.27 1.27)) (justify left top))
+    )
+    (instances
+      (project "_HW_EPaper"
+        (path "/adfaa0ae-c952-44c7-bc24-1bfe8f9a84a3" (page "12"))
+      )
     )
   )

Commit message: Latest update
Other:
- note added: "BATTERY CIRCUIT"
- note added: "BLOCK DIAGRAM"
- note added: "DISPLAY DRIVER"
- note added: "INPUT CIRCUIT"
- note added: "LED DRIVER"
- note added: "MCU"
- note added: "MECHANICAL PARTS"
- note added: "PUSH BUTTONS"
- note added: "SERIAL FLASH"
- note added: "SIPO"
- note added: "TEMP SENSOR"
Changed lines of the file:
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@@
     (company "Mend0z0")
     (comment 1 "v1.0")
-    (comment 2 "DRAFT")
+    (comment 2 "PRELIMINARY")
   )
   (polyline (pts (xy 400.05 184.15) (xy 400.05 214.63))
@@
     (fill (type none))
   )
-  (text "REVISION HISTORY" (at 167.64 224.79 0)
+  (text "SERIAL FLASH" (at 50.8 151.13 0)
+    (effects (font (size 4 4)) (justify left bottom))
+  )
+  (text "REVISION HISTORY" (at 165.1 151.13 0)
     (effects (font (size 4 4)) (justify left bottom))
   )
@@
     (effects (font (size 5 5)) (justify left bottom))
   )
+  (text "DISPLAY DRIVER" (at 50.8 189.23 0)
+    (effects (font (size 4 4)) (justify left bottom))
+  )
+  (text "SIPO" (at 50.8 176.53 0)
+    (effects (font (size 4 4)) (justify left bottom))
+  )
   (text "14" (at 140.97 149.86 0)
     (effects (font (size 5 5)) (justify left bottom))
@@
   (text "6" (at 29.21 175.26 0)
     (effects (font (size 5 5)) (justify left bottom))
+  )
+  (text "MCU" (at 50.8 138.43 0)
+    (effects (font (size 4 4)) (justify left bottom))
   )
   (text "9" (at 29.21 213.36 0)
@@
   (text "DRAFT" (at 99.06 83.82 0)
     (effects (font (size 7.62 7.62) italic) (justify left bottom))
+  )
+  (text "INPUT CIRCUIT" (at 50.8 163.83 0)
+    (effects (font (size 4 4)) (justify left bottom))
+  )
+  (text "BATTERY CIRCUIT" (at 50.8 227.33 0)
+    (effects (font (size 4 4)) (justify left bottom))
   )
   (text "Index" (at 50.8 100.33 0)
@@
     (effects (font (size 2.5 2.5)) (justify left bottom))
   )
-  (text "PWR SEQUENCE" (at 167.64 212.09 0)
+  (text "PWR SEQUENCE" (at 165.1 138.43 0)
     (effects (font (size 4 4)) (justify left bottom))
   )
@@
     (effects (font (size 5 5)) (justify left bottom))
   )
+  (text "TEMP SENSOR" (at 50.8 214.63 0)
+    (effects (font (size 4 4)) (justify left bottom))
+  )
   (text "Mark Not Fitted Components as -->\nDifferential Signal Example\nNet Class Example"
     (at 262.89 144.78 0)
@@
     (effects (font (size 1.27 1.27)) (justify left bottom))
   )
+  (text "BLOCK DIAGRAM" (at 50.8 124.46 0)
+    (effects (font (size 4 4)) (justify left bottom))
+  )
+  (text "MECHANICAL PARTS" (at 165.1 124.46 0)
+    (effects (font (size 4 4)) (justify left bottom))
+  )
   (text "LAYOUT NOTE:" (at 373.38 191.77 0)
     (effects (font (size 1.8 1.8) bold) (justify left bottom))
@@
   (text "INFO:" (at 259.08 191.77 0)
     (effects (font (size 2 2) (thickness 0.4) bold) (justify left bottom))
+  )
+  (text "PUSH BUTTONS" (at 50.8 201.93 0)
+    (effects (font (size 4 4)) (justify left bottom))
+  )
+  (text "LED DRIVER" (at 165.1 113.03 0)
+    (effects (font (size 4 4)) (justify left bottom))
   )
   (text "20" (at 140.97 226.06 0)
@@
     )
   )
-  (sheet (at 50.8 194.31) (size 63.5 6.35) (fields_autoplaced)
+  (sheet (at 165.1 118.11) (size 63.5 6.35) (fields_autoplaced)
     (stroke (width 0.1524) (type solid))
     (fill (color 0 0 0 0.0000))
-    (property "Sheetname" "MECHANICAL PARTS" (at 50.8 193.5984 0)
+    (property "Sheetname" "MECHANICAL PARTS" (at 165.1 117.3984 0)
       (effects (font (size 1.27 1.27)) (justify left bottom))
     )
-    (property "Sheetfile" "[12] - MECHANICAL PARTS.kicad_sch" (at 50.8 201.2446 0)
+    (property "Sheetfile" "[12] - MECHANICAL PARTS.kicad_sch" (at 165.1 125.0446 0)
       (effects (font (size 1.27 1.27)) (justify left top))
     )

Commit message: Updating Hardware File structures
Other:
- added sheet PWR SEQUENCE ([13] - PWR SEQUENCE.kicad_sch)
- added sheet REVISION HISTORY ([14] - REVISION HISTORY.kicad_sch)
- note added: "${COMMENT2}"
- note added: "21"
- note added: "22"
- note added: "23"
- note added: "24"
- note added: "25"
- note added: "26"
- note added: "27"
- note added: "28"
- note added: "29"
- note added: "30"
- note added: "3D Preview BOTTOM"
- note added: "3D Preview TOP"
- note added: "BATTERY CHARGER"
- note added: "Board Statistics Stackup Info"
- note added: "MICROCONTROLLER"
- note added: "SHOULD BE ADDED AFTER RELEASE"
- note added: "SR (SIPO)"
- note removed: "BATTERY CIRCUIT"
- note removed: "DRAFT"
- note removed: "MCU"
- note removed: "SIPO"
